File: External_connec.kicad_sch (KiCad schematic)
At the start: 16 parts, among them CN1 JST_Battery, J11 CAN_TX, J12 CAN_RX, J13 Conn_01x08, J14 Conn_01x06, J15 Conn_01x10, J16 Conn_01x08, J2 A - B, J21 U2U, J3 H - L, J4 TYPE-C-31-M12_13, J5 EXT_LOAD, J9 Conn_01x06

Commit message: Started ESP routing
Connections:
- net GPIO15: no longer J15.3 (Pin_3)
- net GPIO16: no longer J15.4 (Pin_4)
- net CAN_H renamed CAN_P
- net CAN_L renamed CAN_N
- net RS-485_A renamed RS485_P
- net RS-485_B renamed RS485_N
- no-connect marks 10 -> 12
Changed lines of the file:
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@@
   (no_connect (at 33.655 27.94))
   (no_connect (at 252.095 98.425))
+  (no_connect (at 197.485 57.15))
+  (no_connect (at 197.485 54.61))
   (no_connect (at 147.32 41.275))
   (no_connect (at 89.535 27.94))
@@
     (effects (font (size 1.27 1.27) bold (color 72 0 0 1)) (justify right bottom))
   )
-  (label "CAN_H" (at 89.535 128.905 0) (fields_autoplaced)
+  (label "CAN_P" (at 89.535 128.905 0) (fields_autoplaced)
     (effects (font (size 1.27 1.27) bold (color 0 0 0 1)) (justify left bottom))
   )
@@
     (effects (font (size 1.27 1.27) bold (color 0 0 255 1)) (justify left bottom))
   )
-  (label "RS-485_B" (at 69.215 171.45 180) (fields_autoplaced)
+  (label "RS485_N" (at 69.215 171.45 180) (fields_autoplaced)
     (effects (font (size 1.27 1.27) bold (color 0 0 0 1)) (justify right bottom))
   )
@@
     (effects (font (size 1.27 1.27) bold (color 0 0 255 1)) (justify left bottom))
   )
-  (label "RS-485_A" (at 31.75 132.08 0) (fields_autoplaced)
+  (label "RS485_P" (at 31.75 132.08 0) (fields_autoplaced)
     (effects (font (size 1.27 1.27) bold (color 0 0 0 1)) (justify left bottom))
   )
@@
     (effects (font (size 1.27 1.27) (thickness 0.254) bold (color 0 0 255 1)) (justify left bottom))
   )
-  (label "CAN_H" (at 69.215 173.99 180) (fields_autoplaced)
+  (label "CAN_P" (at 69.215 173.99 180) (fields_autoplaced)
     (effects (font (size 1.27 1.27) bold (color 0 0 0 1)) (justify right bottom))
   )
@@
     (effects (font (size 1.27 1.27) bold (color 0 194 0 1)) (justify right bottom))
   )
-  (label "RS-485_A" (at 69.215 168.91 180) (fields_autoplaced)
+  (label "RS485_P" (at 69.215 168.91 180) (fields_autoplaced)
     (effects (font (size 1.27 1.27) bold (color 0 0 0 1)) (justify right bottom))
   )
   (label "GPIO16" (at 97.155 184.15 180) (fields_autoplaced)
-    (effects (font (size 1.27 1.27) bold (color 72 0 0 1)) (justify right bottom))
-  )
-  (label "GPIO15" (at 197.485 57.15 180) (fields_autoplaced)
     (effects (font (size 1.27 1.27) bold (color 72 0 0 1)) (justify right bottom))
   )
@@
     (effects (font (size 1.27 1.27) bold (color 72 0 0 1)) (justify left bottom))
   )
-  (label "CAN_L" (at 89.535 131.445 0) (fields_autoplaced)
+  (label "CAN_N" (at 89.535 131.445 0) (fields_autoplaced)
     (effects (font (size 1.27 1.27) bold (color 0 0 0 1)) (justify left bottom))
   )
@@
     (effects (font (size 1.27 1.27) (thickness 0.254) bold (color 0 0 255 1)) (justify left bottom))
   )
-  (label "GPIO16" (at 197.485 54.61 180) (fields_autoplaced)
-    (effects (font (size 1.27 1.27) bold (color 72 0 0 1)) (justify right bottom))
-  )
   (label "U2U_TX" (at 160.655 186.69 180) (fields_autoplaced)
     (effects (font (size 1.27 1.27) bold (color 0 0 255 1)) (justify right bottom))
@@
     (effects (font (size 1.27 1.27) bold (color 72 0 0 1)) (justify right bottom))
   )
-  (label "CAN_L" (at 69.215 176.53 180) (fields_autoplaced)
+  (label "CAN_N" (at 69.215 176.53 180) (fields_autoplaced)
     (effects (font (size 1.27 1.27) bold (color 0 0 0 1)) (justify right bottom))
   )
@@
     (effects (font (size 1.27 1.27) bold (color 72 0 0 1)) (justify right bottom))
   )
-  (label "RS-485_B" (at 31.75 129.54 0) (fields_autoplaced)
+  (label "RS485_N" (at 31.75 129.54 0) (fields_autoplaced)
     (effects (font (size 1.27 1.27) bold (color 0 0 0 1)) (justify left bottom))
   )
@@
     (effects (font (size 1.27 1.27) (thickness 0.254) bold (color 72 0 72 1)) (justify right))
   )
-  (hierarchical_label "CAN_L" (shape input) (at 53.34 176.53 180) (fields_autoplaced)
+  (hierarchical_label "CAN_N" (shape input) (at 53.34 176.53 180) (fields_autoplaced)
     (effects (font (size 1.27 1.27) bold (color 0 0 0 1)) (justify right))
   )
@@
     (effects (font (size 1.27 1.27) (thickness 0.254) bold (color 72 0 72 1)) (justify right))
   )
-  (hierarchical_label "RS-485_A" (shape input) (at 53.34 168.91 180) (fields_autoplaced)
+  (hierarchical_label "RS485_P" (shape input) (at 53.34 168.91 180) (fields_autoplaced)
     (effects (font (size 1.27 1.27) bold (color 0 0 0 1)) (justify right))
   )
@@
     (effects (font (size 1.27 1.27) (thickness 0.254) bold (color 132 132 0 1)) (justify right))
   )
-  (hierarchical_label "RS-485_B" (shape input) (at 53.34 171.45 180) (fields_autoplaced)
+  (hierarchical_label "RS485_N" (shape input) (at 53.34 171.45 180) (fields_autoplaced)
     (effects (font (size 1.27 1.27) bold (color 0 0 0 1)) (justify right))
   )
@@
     (effects (font (size 1.27 1.27) (thickness 0.254) bold (color 0 0 255 1)) (justify right))
   )
-  (hierarchical_label "CAN_H" (shape input) (at 53.34 173.99 180) (fields_autoplaced)
+  (hierarchical_label "CAN_P" (shape input) (at 53.34 173.99 180) (fields_autoplaced)
     (effects (font (size 1.27 1.27) bold (color 0 0 0 1)) (justify right))
   )
