File: Selection_jumpers.kicad_sch (KiCad schematic)
At the start: 7 parts, among them J10 U2RS485_TX, J10 U2U_TX, J17 U2RS485_DE_~{RE}, J17 U2RS485_RX, J17 U2U_RX, J6 R4_TX, J7 R4_RX

Commit message: Added HW-Tinkerers logo and supporting graphics
Other:
- company: (none) -> HW-TINKERERS (hw.tinkerers@gmail.com)
- title: (none) -> HARDWARE TINKERERS ESP32-S3 DB
Changed lines of the file:
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@@
 (kicad_sch (version 20230121) (generator eeschema)
   (paper "A4")
+  (title_block
+    (title "HARDWARE TINKERERS ESP32-S3 DB")
+    (rev "1.0.0")
+    (company "HW-TINKERERS (hw.tinkerers@gmail.com)")
+    (comment 1 "Email: bhandarkasrishtikr111@gmail.com")
+    (comment 2 "Author: Srishtik Bhandarkar")
+    (comment 3 "Email: vaibhavkhatri00@gmail.com")
+    (comment 4 "Author: Vaibhav Khatri")
+    (comment 5 "Official HW-Tinkerers email: hw.tinkerers@gmail.com")
+  )
   (junction (at 120.65 82.55) (diameter 0) (color 0 0 0 0)
   )
