File: 3V3_Power.kicad_sch (KiCad schematic)
At the start: 8 parts, among them U5 LD1117DT33CTR

Commit message: Added HW-Tinkerers logo and supporting graphics
Other:
- company: (none) -> HW-TINKERERS (hw.tinkerers@gmail.com)
- title: (none) -> HARDWARE TINKERERS ESP32-S3 DB
Changed lines of the file:
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@@
 (kicad_sch (version 20230121) (generator eeschema)
   (paper "A4")
+  (title_block
+    (title "HARDWARE TINKERERS ESP32-S3 DB")
+    (rev "1.0.0")
+    (company "HW-TINKERERS (hw.tinkerers@gmail.com)")
+    (comment 1 "Email: bhandarkasrishtikr111@gmail.com")
+    (comment 2 "Author: Srishtik Bhandarkar")
+    (comment 3 "Email: vaibhavkhatri00@gmail.com")
+    (comment 4 "Author: Vaibhav Khatri")
+    (comment 5 "Official HW-Tinkerers email: hw.tinkerers@gmail.com")
+  )
   (junction (at 189.865 89.535) (diameter 0) (color 0 0 0 0)
   )

Commit message: Added production files for JLC (BOM and CPL)
Parts:
- C16: LCSC Part Number (none) -> C14664
- C17, C42, C43, C44: LCSC Part Number (none) -> C15850
- R22, R23: LCSC Part Number (none) -> C95177
- U5: LCSC Part Number (none) -> C36395
Changed lines of the file:
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@@
+      (effects (font (size 1.27 1.27)) hide)
+    )
+    (property "LCSC Part Number" "C14664" (at 131.445 97.155 0)
       (effects (font (size 1.27 1.27)) hide)
     )
@@
     )
     (property "PN" "CL21A106KAYNNNE" (at 189.865 94.615 0)
+      (effects (font (size 1.27 1.27)) hide)
+    )
+    (property "LCSC Part Number" "C15850" (at 189.865 94.615 0)
       (effects (font (size 1.27 1.27)) hide)
     )
@@
       (effects (font (size 1.27 1.27)) hide)
     )
+    (property "LCSC Part Number" "C36395" (at 146.685 86.36 0)
+      (effects (font (size 1.27 1.27)) hide)
+    )
     (pin "1")
     (pin "2")
@@
       (effects (font (size 1.27 1.27)) hide)
     )
+    (property "LCSC Part Number" "C95177" (at 125.73 89.535 0)
+      (effects (font (size 1.27 1.27)) hide)
+    )
     (pin "1")
     (pin "2")
@@
     )
     (property "PN" "CL21A106KAYNNNE" (at 163.195 94.615 0)
+      (effects (font (size 1.27 1.27)) hide)
+    )
+    (property "LCSC Part Number" "C15850" (at 163.195 94.615 0)
       (effects (font (size 1.27 1.27)) hide)
     )
@@
       (effects (font (size 1.27 1.27)) hide)
     )
+    (property "LCSC Part Number" "C95177" (at 194.945 89.535 0)
+      (effects (font (size 1.27 1.27)) hide)
+    )
     (pin "1")
     (pin "2")
@@
       (effects (font (size 1.27 1.27)) hide)
     )
+    (property "LCSC Part Number" "C15850" (at 180.975 94.615 0)
+      (effects (font (size 1.27 1.27)) hide)
+    )
     (pin "1")
     (pin "2")
@@
       (effects (font (size 1.27 1.27)) hide)
     )
+    (property "LCSC Part Number" "C15850" (at 172.085 94.615 0)
+      (effects (font (size 1.27 1.27)) hide)
+    )
