File: PCB_Attributes.kicad_sch (KiCad schematic)
At the start: 5 parts

Commit message: Added production files for JLC (BOM and CPL)
Parts:
- H1, H2, H3: now left out of the parts list
Changed lines of the file:
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@@
   )
   (symbol (lib_id "ESP32-S3_DB:MountingHole") (at 80.645 64.135 0) (unit 1)
-    (in_bom yes) (on_board yes) (dnp no)
+    (in_bom no) (on_board yes) (dnp no)
     (property "Reference" "H1" (at 79.375 60.96 0)
       (effects (font (size 1.27 1.27)) (justify left))
@@
     )
     (property "Datasheet" "~" (at 80.645 64.135 0)
+      (effects (font (size 1.27 1.27)) hide)
+    )
+    (property "Sim.Enable" "0" (at 80.645 64.135 0)
       (effects (font (size 1.27 1.27)) hide)
     )
@@
   )
   (symbol (lib_id "ESP32-S3_DB:MountingHole") (at 85.725 56.515 0) (unit 1)
-    (in_bom yes) (on_board yes) (dnp no)
+    (in_bom no) (on_board yes) (dnp no)
     (property "Reference" "H3" (at 84.455 53.34 0)
       (effects (font (size 1.27 1.27)) (justify left))
@@
     )
     (property "Datasheet" "~" (at 85.725 56.515 0)
+      (effects (font (size 1.27 1.27)) hide)
+    )
+    (property "Sim.Enable" "0" (at 85.725 56.515 0)
       (effects (font (size 1.27 1.27)) hide)
     )
@@
   )
   (symbol (lib_id "ESP32-S3_DB:MountingHole") (at 75.565 56.515 0) (unit 1)
-    (in_bom yes) (on_board yes) (dnp no)
+    (in_bom no) (on_board yes) (dnp no)
     (property "Reference" "H2" (at 74.295 53.34 0)
       (effects (font (size 1.27 1.27)) (justify left))
@@
       (effects (font (size 1.27 1.27)) hide)
     )
+    (property "Sim.Enable" "0" (at 75.565 56.515 0)
+      (effects (font (size 1.27 1.27)) hide)
+    )
