File: SD_Card.kicad_sch (KiCad schematic)
At the start: 5 parts, among them J8 Micro_SD_Card_Det1

Commit message: Added production files for JLC (BOM and CPL)
Parts:
- C29: LCSC Part Number (none) -> C14664
- C30: LCSC Part Number (none) -> C2173920
- D10: LCSC Part Number (none) -> C477992; PN PESD2CAN -> PESD3V3L5UY,115
- J8: LCSC Part Number (none) -> C5333937
- R12: LCSC Part Number (none) -> C95177
Changed lines of the file:
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@@
+      (effects (font (size 1.27 1.27)) hide)
+    )
+    (property "LCSC Part Number" "C95177" (at 175.895 84.455 0)
       (effects (font (size 1.27 1.27)) hide)
     )
@@
     )
     (property "PN" "TF-012-P9" (at 213.995 86.995 0)
+      (effects (font (size 1.27 1.27)) hide)
+    )
+    (property "LCSC Part Number" "C5333937" (at 213.995 86.995 0)
       (effects (font (size 1.27 1.27)) hide)
     )
@@
       (effects (font (size 1.27 1.27)) hide)
     )
+    (property "LCSC Part Number" "C2173920" (at 215.265 114.3 0)
+      (effects (font (size 1.27 1.27)) hide)
+    )
     (pin "1")
     (pin "2")
@@
       (effects (font (size 1.27 1.27)) hide)
     )
+    (property "LCSC Part Number" "C14664" (at 226.695 114.3 0)
+      (effects (font (size 1.27 1.27)) hide)
+    )
     (pin "1")
     (pin "2")
@@
       (effects (font (size 1.27 1.27)) hide)
     )
-    (property "PN" "PESD2CAN" (at 95.885 103.505 0)
+    (property "PN" "PESD3V3L5UY,115" (at 95.885 103.505 0)
       (effects (font (size 1.27 1.27)) hide)
     )
+    (property "LCSC Part Number" "C477992" (at 95.885 103.505 0)
+      (effects (font (size 1.27 1.27)) hide)
+    )
